File: Esp32_AGV_Relay.kicad_sch (KiCad schematic)
At the start: 19 parts, among them J1 Sensor, J2 LCD1602, J3 Barcode Reader, J4 Left, J5 Conn_01x06, J6 Conn_01x06, J7 Reset, J8 right, Q1 BSS138, Q2 BSS138, U1 PC817

Commit message: v2
1. 改成下拉電阻
2. 更換連接器
Parts:
- removed J8: right, Connector_PinSocket_2.54mm:PinSocket_2x02_P2.54mm_Vertical, symbol Connector_Generic:Conn_02x02_Top_Bottom
- removed R2: 1K, Resistor_SMD:R_0805_2012Metric, symbol Device:R_US
- added J8: right, Connector_PinSocket_2.54mm:PinSocket_1x02_P2.54mm_Vertical, symbol Connector_Generic:Conn_01x02
- added R5: 4.7K, Resistor_SMD:R_0805_2012Metric, symbol Device:R_US
- J6: renamed from J1; footprint TerminalBlock_Phoenix:TerminalBlock_Phoenix_MPT-0,5-2-2.54_1x02_P2.54mm_Horizontal -> TerminalBlock_Phoenix:TerminalBlock_Phoenix_MKDS-1,5-2-5.08_1x02_P5.08mm_Horizontal
- renumbered J2 to J1, J5 to J2, J6 to J3, J3 to J4, J4 to J5, R3 to R1, R4 to R2, R1 to R3, R5 to R4
Connections:
- net +3.3V: now also U1.4
- net EN: now also J8.1 (Pin_1)
- net GND: now also R5.1; no longer U1.3
- net IO19: now also U1.3, R5.2; no longer U1.4
